File: pcb/esp32-c3-board/esp32-c3-board-waveshare.kicad_pcb (KiCad board)
At the start: 2 copper layers, 118.7 x 40.6 mm, 30 parts, among them P101 CAN, P102 RS485, P3 CONN_1, P4 CONN_1, P5 CONN_1, P6 CONN_1, U1 ESP32-C3-Waveshare, U102 TJA1050, U4 6N137, U5 DCDCConverter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

Commit message: Updated boards and readme
Parts:
- moved R3 0.90 mm to (115.8, 58.9)
Routing:
- net GND: track 178.1 -> 173.6 mm
- net 3v3: track 49.5 -> 52.3 mm
- net 5V BMS: track 24.8 -> 26.4 mm
- net Net-(U4-A): track 2.93 -> 3.77 mm
- net RX from BMS: track 22.8 -> 23.6 mm
